File: pic-dev-board.kicad/ShiftRegister.sch (KiCad schematic (older format))
At the start: 15 parts, among them J10 Jumper, J11 Conn_01x05, J12 Conn_01x08_Male, J13 Jumper, J14 Jumper, U2 74HC595

Commit message: added second shift-register
Parts:
- removed J11: Conn_01x05, Connector_PinHeader_2.54mm:PinHeader_1x05_P2.54mm_Vertical, symbol Connector_Generic:Conn_01x05
- removed J13: Jumper, Connector_PinHeader_2.54mm:PinHeader_1x02_P2.54mm_Vertical, symbol Connector:Conn_01x02_Male
- added D15, D16, D17, D18, D19, D20, D21, D22: LED, LED_THT:LED_D3.0mm, symbol Device:LED
- added J11: Conn_01x08_Male, Connector_PinHeader_2.54mm:PinHeader_1x08_P2.54mm_Vertical, symbol Connector:Conn_01x08_Male
- added RN2: 680, Resistor_THT:R_Array_SIP9, symbol Device:R_Network08
- added U3: 74HC595, Package_DIP:DIP-16_W7.62mm_Socket, symbol 74xx:74HC595
Connections:
- net labels added: SA, SB, SC, SD, SE, SF, SG, SH
- wire segments 82 -> 136
- no-connect marks 0 -> 1
Other:
- note removed: "Vout\nSERout\nSCLKout\nRCLKout\nGND"
- moved on the sheet: D10, D11, D12, D13, D14, D7, D8, D9, J10, J12, J14, RN1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

Commit message: added footprints
Parts:
- D10, D11, D12, D13, D14, D15, D16, D17, D18, D19, D20, D21, D22, D7, D8, D9: footprint LED_THT:LED_D3.0mm -> user:LED_1206_3216_Pad1.7x1.75mm_BB
Changed lines of the file:
@@
 F 0 "D13" H 4350 4600 50  0000 C CNN
 F 1 "LED" H 4200 4600 50  0000 C CNN
-F 2 "LED_THT:LED_D3.0mm" H 4150 4700 50  0001 C CNN
+F 2 "user:LED_1206_3216_Pad1.7x1.75mm_BB" H 4150 4700 50  0001 C CNN
 F 3 "~" H 4150 4700 50  0001 C CNN
 	1    4150 4700
@@
 F 0 "D12" H 4350 4400 50  0000 C CNN
 F 1 "LED" H 4200 4400 50  0000 C CNN
-F 2 "LED_THT:LED_D3.0mm" H 4150 4500 50  0001 C CNN
+F 2 "user:LED_1206_3216_Pad1.7x1.75mm_BB" H 4150 4500 50  0001 C CNN
 F 3 "~" H 4150 4500 50  0001 C CNN
 	1    4150 4500
@@
 F 0 "D11" H 4350 4150 50  0000 C CNN
 F 1 "LED" H 4200 4150 50  0000 C CNN
-F 2 "LED_THT:LED_D3.0mm" H 4150 4250 50  0001 C CNN
+F 2 "user:LED_1206_3216_Pad1.7x1.75mm_BB" H 4150 4250 50  0001 C CNN
 F 3 "~" H 4150 4250 50  0001 C CNN
 	1    4150 4250
@@
 F 0 "D10" H 4350 3900 50  0000 C CNN
 F 1 "LED" H 4200 3900 50  0000 C CNN
-F 2 "LED_THT:LED_D3.0mm" H 4150 4000 50  0001 C CNN
+F 2 "user:LED_1206_3216_Pad1.7x1.75mm_BB" H 4150 4000 50  0001 C CNN
 F 3 "~" H 4150 4000 50  0001 C CNN
 	1    4150 4000
@@
 F 0 "D9" H 4350 3650 50  0000 C CNN
 F 1 "LED" H 4200 3650 50  0000 C CNN
-F 2 "LED_THT:LED_D3.0mm" H 4150 3750 50  0001 C CNN
+F 2 "user:LED_1206_3216_Pad1.7x1.75mm_BB" H 4150 3750 50  0001 C CNN
 F 3 "~" H 4150 3750 50  0001 C CNN
 	1    4150 3750
@@
 F 0 "D8" H 4350 3400 50  0000 C CNN
 F 1 "LED" H 4200 3400 50  0000 C CNN
-F 2 "LED_THT:LED_D3.0mm" H 4150 3500 50  0001 C CNN
+F 2 "user:LED_1206_3216_Pad1.7x1.75mm_BB" H 4150 3500 50  0001 C CNN
 F 3 "~" H 4150 3500 50  0001 C CNN
 	1    4150 3500
@@
 F 0 "D14" H 4350 4850 50  0000 C CNN
 F 1 "LED" H 4200 4850 50  0000 C CNN
-F 2 "LED_THT:LED_D3.0mm" H 4150 4950 50  0001 C CNN
+F 2 "user:LED_1206_3216_Pad1.7x1.75mm_BB" H 4150 4950 50  0001 C CNN
 F 3 "~" H 4150 4950 50  0001 C CNN
 	1    4150 4950
@@
 F 0 "D7" H 4350 3150 50  0000 C CNN
 F 1 "LED" H 4200 3150 50  0000 C CNN
-F 2 "LED_THT:LED_D3.0mm" H 4150 3250 50  0001 C CNN
+F 2 "user:LED_1206_3216_Pad1.7x1.75mm_BB" H 4150 3250 50  0001 C CNN
 F 3 "~" H 4150 3250 50  0001 C CNN
 	1    4150 3250
@@
 F 0 "D21" H 9400 4600 50  0000 C CNN
 F 1 "LED" H 9250 4600 50  0000 C CNN
-F 2 "LED_THT:LED_D3.0mm" H 9200 4700 50  0001 C CNN
+F 2 "user:LED_1206_3216_Pad1.7x1.75mm_BB" H 9200 4700 50  0001 C CNN
 F 3 "~" H 9200 4700 50  0001 C CNN
 	1    9200 4700
@@
 F 0 "D20" H 9400 4400 50  0000 C CNN
 F 1 "LED" H 9250 4400 50  0000 C CNN
-F 2 "LED_THT:LED_D3.0mm" H 9200 4500 50  0001 C CNN
+F 2 "user:LED_1206_3216_Pad1.7x1.75mm_BB" H 9200 4500 50  0001 C CNN
 F 3 "~" H 9200 4500 50  0001 C CNN
 	1    9200 4500
@@
 F 0 "D19" H 9400 4150 50  0000 C CNN
 F 1 "LED" H 9250 4150 50  0000 C CNN
-F 2 "LED_THT:LED_D3.0mm" H 9200 4250 50  0001 C CNN
+F 2 "user:LED_1206_3216_Pad1.7x1.75mm_BB" H 9200 4250 50  0001 C CNN
 F 3 "~" H 9200 4250 50  0001 C CNN
 	1    9200 4250
@@
 F 0 "D18" H 9400 3900 50  0000 C CNN
 F 1 "LED" H 9250 3900 50  0000 C CNN
-F 2 "LED_THT:LED_D3.0mm" H 9200 4000 50  0001 C CNN
+F 2 "user:LED_1206_3216_Pad1.7x1.75mm_BB" H 9200 4000 50  0001 C CNN
 F 3 "~" H 9200 4000 50  0001 C CNN
 	1    9200 4000
@@
 F 0 "D17" H 9400 3650 50  0000 C CNN
 F 1 "LED" H 9250 3650 50  0000 C CNN
-F 2 "LED_THT:LED_D3.0mm" H 9200 3750 50  0001 C CNN
+F 2 "user:LED_1206_3216_Pad1.7x1.75mm_BB" H 9200 3750 50  0001 C CNN
 F 3 "~" H 9200 3750 50  0001 C CNN
 	1    9200 3750
@@
 F 0 "D16" H 9400 3400 50  0000 C CNN
 F 1 "LED" H 9250 3400 50  0000 C CNN
-F 2 "LED_THT:LED_D3.0mm" H 9200 3500 50  0001 C CNN
+F 2 "user:LED_1206_3216_Pad1.7x1.75mm_BB" H 9200 3500 50  0001 C CNN
 F 3 "~" H 9200 3500 50  0001 C CNN
 	1    9200 3500
@@
 F 0 "D22" H 9400 4850 50  0000 C CNN
 F 1 "LED" H 9250 4850 50  0000 C CNN
-F 2 "LED_THT:LED_D3.0mm" H 9200 4950 50  0001 C CNN
+F 2 "user:LED_1206_3216_Pad1.7x1.75mm_BB" H 9200 4950 50  0001 C CNN
 F 3 "~" H 9200 4950 50  0001 C CNN
 	1    9200 4950
@@
 F 0 "D15" H 9400 3150 50  0000 C CNN
 F 1 "LED" H 9250 3150 50  0000 C CNN
-F 2 "LED_THT:LED_D3.0mm" H 9200 3250 50  0001 C CNN
+F 2 "user:LED_1206_3216_Pad1.7x1.75mm_BB" H 9200 3250 50  0001 C CNN
 F 3 "~" H 9200 3250 50  0001 C CNN
 	1    9200 3250

Commit message: changed values of connectors
Parts:
- J10: value Jumper -> Jumper DATin
- J11: value Conn_01x08_Male -> Conn_SR_2
- J12: value Conn_01x08_Male -> Conn_SR_1
- J14: value Jumper -> Jumper CLKin
Changed lines of the file:
@@
 P 4950 5650
 F 0 "J12" V 4877 5578 50  0000 C CNN
-F 1 "Conn_01x08_Male" V 4786 5578 50  0000 C CNN
+F 1 "Conn_SR_1" V 4786 5578 50  0000 C CNN
 F 2 "Connector_PinHeader_2.54mm:PinHeader_1x08_P2.54mm_Vertical" H 4950 5650 50  0001 C CNN
 F 3 "~" H 4950 5650 50  0001 C CNN
@@
 P 1700 2400
 F 0 "J10" H 1600 2350 50  0000 C CNN
-F 1 "Jumper" H 1600 2250 50  0000 C CNN
+F 1 "Jumper DATin" H 1600 2250 50  0000 C CNN
 F 2 "Connector_PinHeader_2.54mm:PinHeader_1x02_P2.54mm_Vertical" H 1700 2400 50  0001 C CNN
 F 3 "~" H 1700 2400 50  0001 C CNN
@@
 P 1600 2900
 F 0 "J14" H 1500 2850 50  0000 C CNN
-F 1 "Jumper" H 1500 2750 50  0000 C CNN
+F 1 "Jumper CLKin" H 1500 2750 50  0000 C CNN
 F 2 "Connector_PinHeader_2.54mm:PinHeader_1x02_P2.54mm_Vertical" H 1600 2900 50  0001 C CNN
 F 3 "~" H 1600 2900 50  0001 C CNN
@@
 P 10050 5650
 F 0 "J11" V 9977 5578 50  0000 C CNN
-F 1 "Conn_01x08_Male" V 9886 5578 50  0000 C CNN
+F 1 "Conn_SR_2" V 9886 5578 50  0000 C CNN
 F 2 "Connector_PinHeader_2.54mm:PinHeader_1x08_P2.54mm_Vertical" H 10050 5650 50  0001 C CNN
 F 3 "~" H 10050 5650 50  0001 C CNN
