File: pic-dev-board.kicad/pic-dev-board.kicad_pcb (KiCad board)
At the start: 2 copper layers, 100 x 100 mm, 80 parts, among them J1 Conn_GP0, J10 Jumper DATin, J11 Conn_SR_2, J12 Conn_SR_1, J13 Conn_5V_GND, J14 Jumper CLKin, J15 Barrel_Jack_Switch, J16 RUN/~PGM, J17 I2C, J18 GP1(RA1)/RB6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

Commit message: added JLC-number field
Other:
- board text added: "JLCJLCJLCJLC"
Changed lines of the file:
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@@
   (general
     (thickness 1.6)
-    (drawings 100)
+    (drawings 101)
     (tracks 695)
     (zones 0)
@@
     )
   )
+  (gr_text JLCJLCJLCJLC (at 108.4326 34.29) (layer F.SilkS)
+    (effects (font (size 1 1) (thickness 0.15)))
+  )
   (gr_text "D7\n-\nD14" (at 69.215 71.7296) (layer F.SilkS)

Commit message: bugfix: labels for GP4/GP5 had CLK/DAT swapped
Other:
- board text added: "CLK (GP5)"
- board text added: "DAT (GP4)"
- board text removed: "CLK (GP4)"
- board text removed: "DAT (GP5)"
